Commit message: fix: syntax error

File: end_effectors/common/franka_hand.xacro (robot description, xacro)
@@ -2,5 +2,17 @@
 <robot xmlns:xacro="http://www.ros.org/wiki/xacro" name="hand">
   <!-- safety_distance: Minimum safety distance in [m] by which the collision volumes are expanded and which is enforced during robot motions -->
-  <xacro:macro name="franka_hand" params="connected_to:='' arm_id arm_prefix:='' ee_id ee_inertials rpy_ee:='0 0 0' xyz_ee:='0 0 0' tcp_xyz:='0 0 0.1034' tcp_rpy:='0 0 0' safety_distance:=0 gazebo:=false description_pkg:=franka_description with_sc:=false">
+  <xacro:macro name="franka_hand"
+               params="connected_to:=''
+                       arm_id arm_prefix:=''
+                       ee_id ee_inertials
+                       rpy_ee:='0 0 0'
+                       xyz_ee:='0 0 0'
+                       tcp_xyz:='0 0 0.1034'
+                       tcp_rpy:='0 0 0'
+                       safety_distance:=0
+                       gazebo:=false
+                       description_pkg:=franka_description
+                       with_sc:=false
+                       no_prefix:=false">
     <xacro:property name="ee_prefix" default="robot_"/>
     <xacro:unless value="${arm_id == ''}">

File: robots/common/franka_arm.ros2_control.xacro (robot description, xacro)
@@ -3,11 +3,12 @@
 <xacro:macro name="franka_arm_ros2_control"
          params="arm_id
-             robot_ip
-             use_fake_hardware:=^|false
-             fake_sensor_commands:=^|false
-             gazebo:=^|false
-             hand:=^|false
-             gazebo_effort:=^|false
-             arm_prefix:=''">
+                 robot_ip
+                 use_fake_hardware:=false
+                 fake_sensor_commands:=false
+                 gazebo:=false
+                 hand:=false
+                 gazebo_effort:=false
+                 arm_prefix:=''
+                 multi_arm:=false">
     <xacro:property name="arm_prefix_modified" value="${'' if arm_prefix == '' else arm_prefix + '_'}" />
     <ros2_control name="${arm_prefix_modified}FrankaHardwareInterface" type="system">
@@ -51,11 +52,11 @@
         </joint>
       </xacro:macro>
-      <xacro:configure_joint joint_name="${arm_prefix_modified}${arm_id}_joint1" initial_position="0.0"/>
-      <xacro:configure_joint joint_name="${arm_prefix_modified}${arm_id}_joint2" initial_position="${-pi/4}"/>
-      <xacro:configure_joint joint_name="${arm_prefix_modified}${arm_id}_joint3" initial_position="0.0"/>
-      <xacro:configure_joint joint_name="${arm_prefix_modified}${arm_id}_joint4" initial_position="${-3*pi/4}"/>
-      <xacro:configure_joint joint_name="${arm_prefix_modified}${arm_id}_joint5" initial_position="0.0"/>
-      <xacro:configure_joint joint_name="${arm_prefix_modified}${arm_id}_joint6" initial_position="${pi/2}"/>
-      <xacro:configure_joint joint_name="${arm_prefix_modified}${arm_id}_joint7" initial_position="${pi/4}"/>
+      <xacro:configure_joint joint_name="${arm_prefix}${arm_id}_joint1" initial_position="0.0"/>
+      <xacro:configure_joint joint_name="${arm_prefix}${arm_id}_joint2" initial_position="${-pi/4}"/>
+      <xacro:configure_joint joint_name="${arm_prefix}${arm_id}_joint3" initial_position="0.0"/>
+      <xacro:configure_joint joint_name="${arm_prefix}${arm_id}_joint4" initial_position="${-3*pi/4}"/>
+      <xacro:configure_joint joint_name="${arm_prefix}${arm_id}_joint5" initial_position="0.0"/>
+      <xacro:configure_joint joint_name="${arm_prefix}${arm_id}_joint6" initial_position="${pi/2}"/>
+      <xacro:configure_joint joint_name="${arm_prefix}${arm_id}_joint7" initial_position="${pi/4}"/>
       <xacro:if value="${gazebo and hand}">
         <xacro:configure_joint joint_name="${arm_id}_finger_joint1" initial_position="0.0" />

File: robots/common/franka_robot.xacro (robot description, xacro)
@@ -10,4 +10,9 @@
                       xyz:='0 0 0'
                       rpy:='0 0 0'
+                      xyz_ee:='0 0 0'
+                      rpy_ee:='0 0 0'
+                      tcp_xyz:='0 0 0'
+                      tcp_rpy:='0 0 0'
+                      safety_distance:='0.03'
                       hand:='true'
                       ee_id:=none
@@ -24,8 +29,7 @@
     <xacro:include filename="$(find franka_description)/robots/common/utils.xacro" />
     <xacro:include filename="$(find franka_description)/robots/common/franka_arm.xacro" />
-    <xacro:property name="arm_prefix_modified" value="${'' if arm_prefix == '' else arm_prefix + '_'}" />
     <xacro:franka_arm
       arm_id="${arm_id}"
-      arm_prefix="${arm_prefix_modified}"
+      arm_prefix="${arm_prefix}"
       no_prefix="${no_prefix}"
       xyz="${xyz}"
@@ -43,5 +47,5 @@
       <xacro:include filename="$(find franka_description)/end_effectors/common/franka_hand.xacro"/>
       <xacro:include filename="$(find franka_description)/end_effectors/common/utils.xacro" />
-      <xacro:include filename="$(find franka_description)/end_effectors/$(arg ee_id)/$(arg ee_id)_arguments.xacro" />
+      <xacro:include filename="$(find franka_description)/end_effectors/${ee_id}/${ee_id}_arguments.xacro" />
       <xacro:if value="${arm_id == 'fp3'}">
         <xacro:property name="ee_color" value="black" />
@@ -53,14 +57,14 @@
       <xacro:property name="connection" value="${special_connection if special_connection != '' else arm_id + '_link8'}" />
       <xacro:franka_hand
-        connected_to="${arm_prefix_modified}${connection}"
+        connected_to="${arm_prefix}${connection}"
         arm_id="${arm_id}"
-        arm_prefix="${arm_prefix_modified}"
+        arm_prefix="${arm_prefix}"
         ee_id="${ee_id}_${ee_color}"
-        ee_inertials="${xacro.load_yaml('$(find franka_description)/end_effectors/$(arg ee_id)/inertials.yaml')}"
-        rpy_ee="$(arg rpy_ee)"
-        xyz_ee="$(arg xyz_ee)"
-        tcp_xyz="$(arg tcp_xyz)"
-        tcp_rpy="$(arg tcp_rpy)"
-        safety_distance="$(arg safety_distance)"
+        ee_inertials="${xacro.load_yaml('$(find franka_description)/end_effectors/' + ee_id + '/inertials.yaml')}"
+        rpy_ee="${rpy_ee}"
+        xyz_ee="${xyz_ee}"
+        tcp_xyz="${tcp_xyz}"
+        tcp_rpy="${tcp_rpy}"
+        safety_distance="${safety_distance}"
         gazebo="${gazebo}"
         description_pkg="$(arg description_pkg)"
@@ -71,18 +75,18 @@
       <xacro:include filename="$(find franka_description)/end_effectors/common/ee_with_one_link.xacro"/>
       <xacro:include filename="$(find franka_description)/end_effectors/common/utils.xacro" />
-      <xacro:include filename="$(find franka_description)/end_effectors/$(arg ee_id)/$(arg ee_id)_arguments.xacro" />
-      <xacro:property name="special_connection" value="$(arg special_connection)" />
+      <xacro:include filename="$(find franka_description)/end_effectors/' + ee_id + '/' + ee_id + '_arguments.xacro" />
+      <xacro:property name="special_connection" value="${special_connection}" />
       <xacro:property name="connection" value="${special_connection if special_connection == '' else arm_id + '_link8'}" />
       <xacro:ee_with_one_link
-        connected_to="${arm_prefix_modified}${connection}"
+        connected_to="${arm_prefix}${connection}"
         arm_id="${arm_id}"
-        arm_prefix="${arm_prefix_modified}"
+        arm_prefix="${arm_prefix}"
         ee_id="${ee_id}"
-        ee_inertials="${xacro.load_yaml('$(find franka_description)/end_effectors/$(arg ee_id)/inertials.yaml')}"
-        rpy_ee="$(arg rpy_ee)"
-        xyz_ee="$(arg xyz_ee)"
-        tcp_xyz="$(arg tcp_xyz)"
-        tcp_rpy="$(arg tcp_rpy)"
-        safety_distance="$(arg safety_distance)"
+        ee_inertials="${xacro.load_yaml('$(find franka_description)/end_effectors/${ee_id}/inertials.yaml')}"
+        rpy_ee="${rpy_ee}"
+        xyz_ee="${xyz_ee}"
+        tcp_xyz="${tcp_xyz}"
+        tcp_rpy="${tcp_rpy}"
+        safety_distance="${safety_distance}"
         gazebo="${gazebo}"
         description_pkg="$(arg description_pkg)"
@@ -142,9 +146,9 @@
           arm_id="${arm_id}"
           robot_ip="${robot_ip}"
-          use_fake_hardware="$(arg use_fake_hardware)"
-          fake_sensor_commands="$(arg fake_sensor_commands)"
-          gazebo="$(arg gazebo)"
-          hand="$(arg hand)"
-          gazebo_effort="$(arg gazebo_effort)"
+          use_fake_hardware="${use_fake_hardware}"
+          fake_sensor_commands="${fake_sensor_commands}"
+          gazebo="${gazebo}"
+          hand="${hand}"
+          gazebo_effort="${gazebo_effort}"
           arm_prefix="${arm_prefix}"
       />

File: robots/fr3/fr3.urdf.xacro (robot description, xacro)
@@ -50,5 +50,5 @@
                       gazebo_effort="$(arg gazebo_effort)"
                       no_prefix="$(arg no_prefix)"
-                      arm_prefix="$(arg arm_prefix)"
+                      arm_prefix="${modified_prefix}"
                       connected_to= "base">
   </xacro:franka_robot>

File: robots/fr3_duo/fr3_duo.urdf.xacro (robot description, xacro)
@@ -49,4 +49,5 @@
       <xacro:property name="mount_to_base" value="${xacro.load_yaml('$(arg mount_kinematics)')}"/>
       <xacro:property name="robot_prefix" value="${arm_prefixes_list[i]}"/>
+      <xacro:property name="modified_prefix" value="${robot_prefix + '_' if robot_prefix else ''}"/>
       <joint name="${arm_prefixes_list[i]}_base_joint" type="fixed">
         <parent link="mount_link"/>
@@ -80,5 +81,5 @@
                           gazebo_effort="$(arg gazebo_effort)"
                           no_prefix="$(arg no_prefix)"
-                          arm_prefix= "${arm_prefixes_list[i]}"
+                          arm_prefix= "${modified_prefix}"
                           connected_to="${arm_prefixes_list[i]}_base">
       </xacro:franka_robot>

File: robots/fr3_duo/fr3_duo_arm.urdf.xacro (robot description, xacro)
@@ -32,4 +32,7 @@
   <!-- Should the robot be spawned in Gazebo with effort interfaces?" -->
   <xacro:arg name="gazebo_effort" default="false" />
+  <!-- Append an underscore to the user-provided prefix, if non-empty. -->
+  <xacro:property name="prefix" value="$(arg arm_prefix)"/>
+  <xacro:property name="modified_prefix" value="${prefix + '_' if prefix else ''}"/>
   <link name="base">
   </link>
@@ -68,5 +71,5 @@
                       gazebo_effort="$(arg gazebo_effort)"
                       no_prefix="$(arg no_prefix)"
-                      arm_prefix= "${arm_prefix_i}"
+                      arm_prefix= "${modified_prefix}"
                       connected_to="${arm_prefix_i}_base">
       </xacro:franka_robot>

File: robots/fr3v2/fr3v2.urdf.xacro (robot description, xacro)
@@ -8,4 +8,6 @@
   -->
   <xacro:arg name="arm_id" default="fr3v2" />
+  <!-- The prefix of the robot -->
+  <xacro:arg name="arm_prefix" default="" />
   <!-- Don't print a prefix for joints, visuals, and links? -->
   <xacro:arg name="no_prefix" default="false"/>
@@ -28,4 +30,7 @@
   <!-- Should the robot be spawned in Gazebo with effort interfaces?" -->
   <xacro:arg name="gazebo_effort" default="false" />
+  <!-- Append an underscore to the user-provided prefix, if non-empty. -->
+  <xacro:property name="prefix" value="$(arg arm_prefix)"/>
+  <xacro:property name="modified_prefix" value="${prefix + '_' if prefix else ''}"/>
   <xacro:franka_robot arm_id="fr3v2"
                       joint_limits="${xacro.load_yaml('$(find franka_description)/robots/fr3v2/joint_limits.yaml')}"
@@ -43,5 +48,5 @@
                       gazebo_effort="$(arg gazebo_effort)"
                       no_prefix="$(arg no_prefix)"
-                      arm_prefix= ""
+                      arm_prefix= "${modified_prefix}"
                       connected_to= "base">
   </xacro:franka_robot>
