Commit message: fix: cover and mount replaced by new designs

File: robots/fr3_duo/fr3_duo_mount/fr3_duo_mount.xacro (robot description, xacro)
@@ -6,9 +6,6 @@
       <visual>
         <geometry>
-          <mesh filename="package://franka_description/meshes/robot_arms/fr3_duo/mount/visual/fr3_duo_mount.stl"/>
+          <mesh filename="package://franka_description/meshes/robot_arms/fr3_duo/mount/visual/fr3_duo_mount.dae"/>
         </geometry>
-        <material name="white">
-          <color rgba="0.5 0.5 0.5 1.0" />
-        </material>
       </visual>
       <collision>
