Commit message: replace _ with /

File: robots/fr3/fr3.urdf.xacro (robot description, xacro)
@@ -46,5 +46,5 @@
   <!-- Append an underscore to the user-provided prefix, if non-empty. -->
   <xacro:property name="prefix" value="$(arg arm_prefix)"/>
-  <xacro:property name="modified_prefix" value="${prefix + '_' if prefix else ''}"/>
+  <xacro:property name="modified_prefix" value="${prefix + '/' if prefix else ''}"/>
   <xacro:franka_robot arm_id="fr3"
                       joint_limits="${xacro.load_yaml('$(find franka_description)/robots/fr3/joint_limits.yaml')}"
